File: KiCad-design/A2 audio helper.kicad_sch (KiCad schematic)
At the start: 35 parts, among them J1 PIN HEADER 1x2, J10 PIN HEADER 1x2, J11 PIN HEADER 1x3, J12 PIN HEADER 1x3, J13 PIN HEADER 2x4, J15 PIN HEADER 2x6, J2 PIN HEADER 1x2, J3 PIN HEADER 1x2, J4 SJ1-3515N, J5 PIN HEADER 1x3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

Commit message: lengthened, new bigger switch part, cleanup
Parts:
- removed SW2: SW_DPDT_x2, Button_Switch_THT:SW_CK_JS202011CQN_DPDT_Straight, symbol Switch:SW_DPDT_x2
- added SW1: EG2209, EG2209:EG2209, symbol EG2209:EG2209
- J1: value PIN HEADER 1x2 -> S2B-XH-A
- J10, J9: value PIN HEADER 1x2 -> AE-6410-2A
- J13: value PIN HEADER 2x4 -> JST B8B-PHDSS
- J3: value PIN HEADER 1x2 -> 22053021
Connections:
- net SPKR_L: now also SW1.3
- net SPKR_R: now also SW1.4
- net at R10.1: now also SW1.6
- net at U1.7 (R+): now also SW1.5
- net at U1.8 (L+): now also SW1.2
- net at R9.1: now also SW1.1
Other:
- note added: "left"
- note removed: "left/mono"
- moved on the sheet: J9, R10, R9
